File: ruecklicht.kicad_pcb (KiCad board)
At the start: 2 copper layers, 67 x 46 mm, 3 parts

Commit message: 15.11.2025 16:38
Parts:
- added B1+1: Conn_01x01_Pin, Connector_Wire:SolderWire-1.5sqmm_1x01_D1.7mm_OD3.9mm, F.Cu at (185.8, 71.5)
- added B1-1: Conn_01x01_Pin, Connector_Wire:SolderWire-1.5sqmm_1x01_D1.7mm_OD3.9mm, F.Cu at (128.2, 71.5)
- added B2+1: Conn_01x01_Pin, Connector_Wire:SolderWire-1.5sqmm_1x01_D1.7mm_OD3.9mm, F.Cu at (128.2, 85.0)
- added B2-1: Conn_01x01_Pin, Connector_Wire:SolderWire-1.5sqmm_1x01_D1.7mm_OD3.9mm, F.Cu at (185.8, 85.0)
- added B3+1: Conn_01x01_Pin, Connector_Wire:SolderWire-1.5sqmm_1x01_D1.7mm_OD3.9mm, F.Cu at (185.8, 98.5)
- added B3-1: Conn_01x01_Pin, Connector_Wire:SolderWire-1.5sqmm_1x01_D1.7mm_OD3.9mm, F.Cu at (128.2, 98.5)
- added C1: 22u, Capacitor_SMD:CP_Elec_4x5.4, F.Cu at (219.8, 76.2)
- added C2: C_Small, Capacitor_SMD:C_0805_2012Metric_Pad1.18x1.45mm_HandSolder, F.Cu at (235.2, 63.3)
- added D10: WS2812B, LED_SMD:LED_WS2812B_PLCC4_5.0x5.0mm_P3.2mm, F.Cu at (177.4, 85.1)
- added D11: WS2812B, LED_SMD:LED_WS2812B_PLCC4_5.0x5.0mm_P3.2mm, F.Cu at (137.2, 98.5)
- added D12: WS2812B, LED_SMD:LED_WS2812B_PLCC4_5.0x5.0mm_P3.2mm, F.Cu at (147.2, 98.5)
- added D14: WS2812B, LED_SMD:LED_WS2812B_PLCC4_5.0x5.0mm_P3.2mm, F.Cu at (167.2, 98.5)
- added D15: WS2812B, LED_SMD:LED_WS2812B_PLCC4_5.0x5.0mm_P3.2mm, F.Cu at (177.2, 98.5)
- added D2: WS2812B, LED_SMD:LED_WS2812B_PLCC4_5.0x5.0mm_P3.2mm, F.Cu at (147.5, 71.5)
- added D3: WS2812B, LED_SMD:LED_WS2812B_PLCC4_5.0x5.0mm_P3.2mm, F.Cu at (157.5, 71.5)
- added D4: WS2812B, LED_SMD:LED_WS2812B_PLCC4_5.0x5.0mm_P3.2mm, F.Cu at (167.5, 71.5)
- added D5: WS2812B, LED_SMD:LED_WS2812B_PLCC4_5.0x5.0mm_P3.2mm, F.Cu at (177.4, 71.5)
- added D6: WS2812B, LED_SMD:LED_WS2812B_PLCC4_5.0x5.0mm_P3.2mm, F.Cu at (137.4, 85.0)
- added D8: WS2812B, LED_SMD:LED_WS2812B_PLCC4_5.0x5.0mm_P3.2mm, F.Cu at (157.4, 85.1)
- added D9: WS2812B, LED_SMD:LED_WS2812B_PLCC4_5.0x5.0mm_P3.2mm, F.Cu at (167.4, 85.1)
- added IC1: SN74HCS74QDYYRQ1, footprints:SOP50P326X110-14N, B.Cu at (173.5, 66.8)
- added IC2: TXS0104EDG4, footprints:SOIC127P600X175-14N, F.Cu at (254.0, 52.8)
- added J1: Conn_01x05_Pin, Connector_PinHeader_2.54mm:PinHeader_1x05_P2.54mm_Vertical, F.Cu at (251.7, 87.9)
- added L1: 1.3u, footprints:4310LC132KEC, F.Cu at (175.7, 50.1)
- added Q1: NMOS, Package_TO_SOT_SMD:TO-252-3_TabPin2, F.Cu at (229.7, 64.7)
- added R1: R, Resistor_SMD:R_1206_3216Metric_Pad1.30x1.75mm_HandSolder, F.Cu at (235.4, 68.7)
- added R2: 140k, Resistor_SMD:R_1206_3216Metric_Pad1.30x1.75mm_HandSolder, F.Cu at (218.6, 69.4)
- added R3: 30.9k, Resistor_SMD:R_1206_3216Metric_Pad1.30x1.75mm_HandSolder, F.Cu at (221.9, 69.4)
- added R4: R_Small, Resistor_SMD:R_1206_3216Metric_Pad1.30x1.75mm_HandSolder, F.Cu at (230.9, 111.4)
- added R5: R_Small, Resistor_SMD:R_1206_3216Metric_Pad1.30x1.75mm_HandSolder, F.Cu at (230.9, 114.8)
- added S1: 431256083716, footprints:431256083716, F.Cu at (216.7, 95.4)
- added S2: 431256083716, footprints:431256083716, F.Cu at (230.3, 95.4)
- added U1: ESP32-C3-MINI-1-H4X, footprints:ESP32C3MINI1H4X, F.Cu at (259.3, 98.3)
- added U2: MP2128DT-LF-P, Package_TO_SOT_SMD:SOT-23-5_HandSoldering, F.Cu at (219.4, 63.5)
- moved D13 21.8 mm to (157.2, 98.5), turned to 180 degrees
- moved D1 21.6 mm to (137.4, 71.5), turned to 180 degrees
- moved D7 16.8 mm to (147.4, 85.1), turned to 180 degrees

Commit message: 16.11.2025 13:36 -> Schematic Finished (possible)
Parts:
- added J2: Conn_01x08_Pin, Connector_PinHeader_2.54mm:PinHeader_1x08_P2.54mm_Vertical, F.Cu at (215.0, 125.2)
- L1: moved to B.Cu
- moved L1 28.5 mm to (173.2, 78.5), turned to 0 degrees
- moved IC1 6.00 mm to (167.5, 67.0), turned to 0 degrees
Routing:
- net /LEDs: track 0.00 -> 46.7 mm
- net Net-(D1-DOUT): track 0.00 -> 7.10 mm
- added copper zone on F.Cu, net GND
- added copper zone on F.Cu, net Net-(B1-1-Pin_1)
- added copper zone on F.Cu, net Net-(B2-1-Pin_1)

Commit message: 16.11.2025 16:28 -> began with pcb
Parts:
- C1, C2, J1, J2, R1, R2, R3, R4, R5, U1, U2: moved to B.Cu
- IC2: footprint footprints:SOIC127P600X175-14N -> Package_SO:SOIC-14_3.9x8.7mm_P1.27mm; moved to B.Cu
- Q1: footprint Package_TO_SOT_SMD:TO-252-3_TabPin2 -> footprints:mosfet; moved to B.Cu
- moved J1 95.7 mm to (156.1, 89.5)
- moved IC2 91.8 mm to (163.5, 68.3), turned to 180 degrees
- moved U1 87.0 mm to (172.5, 93.0)
- moved S2 83.0 mm to (152.2, 67.2), turned to 180 degrees
- moved C1 80.6 mm to (139.2, 77.0), turned to 0 degrees
- moved S1 80.5 mm to (141.2, 67.2), turned to 180 degrees
- moved J2 75.6 mm to (142.0, 105.5), turned to -90 degrees
- moved R3 70.4 mm to (151.5, 70.2), turned to 180 degrees
- moved R1 63.4 mm to (173.2, 81.0), turned to -90 degrees
- moved R5 62.3 mm to (169.3, 106.0), turned to 180 degrees
- moved R4 62.2 mm to (169.3, 103.5), turned to 180 degrees
- moved R2 61.3 mm to (157.2, 70.2), turned to 180 degrees
- moved C2 59.8 mm to (175.5, 65.2), turned to 0 degrees
- moved U2 57.6 mm to (163.2, 76.3), turned to -90 degrees
- moved Q1 51.2 mm to (180.1, 77.2), turned to 0 degrees
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Connections:
- D1 pad 1: /LEDs -> /4.5_GEN
- D10 pad 1: /LEDs -> /4.5_GEN
- D11 pad 1: /LEDs -> /4.5_GEN
- D12 pad 1: /LEDs -> /4.5_GEN
- D13 pad 1: /LEDs -> /4.5_GEN
- D14 pad 1: /LEDs -> /4.5_GEN
- D15 pad 1: /LEDs -> /4.5_GEN
- D2 pad 1: /LEDs -> /4.5_GEN
- D3 pad 1: /LEDs -> /4.5_GEN
- D4 pad 1: /LEDs -> /4.5_GEN
- D5 pad 1: /LEDs -> /4.5_GEN
- D6 pad 1: /LEDs -> /4.5_GEN
- D7 pad 1: /LEDs -> /4.5_GEN
- D8 pad 1: /LEDs -> /4.5_GEN
- D9 pad 1: /LEDs -> /4.5_GEN
- IC2 pad 1: 4.5V -> /4.5_GEN
- U1 pad 22: unconnected-(U1-IO8-Pad22) -> /SDA
- U1 pad 23: unconnected-(U1-IO9-Pad23) -> /SCL
- U1 pad 5: unconnected-(U1-IO2-Pad5) -> /D+
- U1 pad 6: unconnected-(U1-IO3-Pad6) -> /BT_EN_3.3
- U1 pad 8: unconnected-(U1-EN-Pad8) -> +3.3V
Routing:
- net /4.5_GEN: track 0.00 -> 231.3 mm, vias 0 -> 6
- net /leds/D2: track 0.00 -> 65.4 mm
- net /leds/D1: track 0.00 -> 63.5 mm
- net /LEDs: track 46.7 -> 0.00 mm
- net /B+: track 0.00 -> 42.3 mm
- net /switches/Q1: track 0.00 -> 14.2 mm
- net Net-(U2-FB): track 0.00 -> 14.1 mm
- net Net-(U2-SW): track 0.00 -> 13.4 mm, vias 0 -> 2
- net +3.3V: track 0.00 -> 11.1 mm
- net Net-(D12-DOUT): track 0.00 -> 7.69 mm
- net Net-(D14-DOUT): track 0.00 -> 7.64 mm
- net Net-(D13-DOUT): track 0.00 -> 7.64 mm
- net Net-(D6-DOUT): track 0.00 -> 7.53 mm
- net Net-(D7-DOUT): track 0.00 -> 7.49 mm
- net Net-(D8-DOUT): track 0.00 -> 7.44 mm
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- added copper zone on B.Cu, net +3.3V
- added copper zone on B.Cu, net /4.5_GEN
- added copper zone on B.Cu, net /B+
- added copper zone on B.Cu, net GND
Other:
- board text added: "GYRO"

Commit message: Finished Rev.1
Parts:
- J2: moved to F.Cu
- moved J2 17.8 mm to (159.8, 105.6)
- moved S2 11.0 mm to (141.2, 67.3)
- moved S1 10.9 mm to (152.1, 67.3)
- moved R5 2.80 mm to (169.3, 103.2)
- moved R4 2.70 mm to (169.4, 106.2)
- moved J1 0.70 mm to (156.1, 90.2)
Connections:
- J1 pad 1: /ESP32/TX -> /ESP32/RX
- J1 pad 2: /ESP32/RX -> /ESP32/TX
- J1 pad 3: /ESP32/EN -> +3.3V
Routing:
- net +3.3V: track 11.1 -> 96.5 mm, vias 0 -> 3
- net /BT_EN_3.3: track 0.00 -> 80.5 mm, vias 0 -> 2
- net /D+: track 0.00 -> 73.1 mm, vias 0 -> 1
- net /switches/BT_EN_Button/NO: track 0.00 -> 46.5 mm, vias 0 -> 1
- net /SDA: track 0.00 -> 43.4 mm, vias 0 -> 2
- net /SCL: track 0.00 -> 42.3 mm
- net /switches/EN_Button/NO: track 0.00 -> 37.6 mm, vias 0 -> 1
- net /ESP32/TX: track 0.00 -> 23.5 mm
- net /ESP32/RX: track 0.00 -> 18.4 mm
- net /B+: track 42.3 -> 60.7 mm, vias 0 -> 3
- net /BT_EN_4.5: track 0.00 -> 11.7 mm
- net GND: track 3.28 -> 11.4 mm, vias 1 -> 14
- net /switches/d-ff/q-inv2: track 0.00 -> 3.83 mm
- net /switches/d-ff/q-inv: track 6.12 -> 4.37 mm
- net /leds/D1: track 63.5 -> 65.1 mm
Other:
- board text added: "INT"
- board text added: "OPT"
- board text added: "RX"
- board text added: "TX"
- board text added: "VCC"

Commit message: stand before gyro change
Parts:
- J2: moved to B.Cu
- moved R2 1.35 mm to (156.6, 71.4)
- moved R3 1.16 mm to (151.3, 71.4)
- moved J1 0.40 mm to (156.1, 89.8)
- turned J2 to 90 degrees
Routing:
- net GND: track 11.4 -> 9.29 mm, vias 14 -> 43
- net +3.3V: track 96.5 -> 98.5 mm
- net /D+: track 73.1 -> 74.2 mm
- net Net-(U2-FB): track 14.1 -> 13.1 mm
- net /4.5_GEN: track 231.6 -> 230.8 mm

Commit message: Finished Rev.1 -> possible order
Parts:
- J2: footprint Connector_PinHeader_2.54mm:PinHeader_1x08_P2.54mm_Vertical -> footprints:mpu6050-self
- moved J1 25.9 mm to (177.3, 104.6)
- moved J2 14.9 mm to (145.0, 103.2)
- moved R4 9.53 mm to (160.9, 101.8)
- moved R5 8.46 mm to (160.9, 104.2)
Connections:
- J1 pad 4: unconnected-(J1-Pin_4-Pad4) -> GND
Routing:
- net /ESP32/RX: track 18.4 -> 37.9 mm
- net /ESP32/TX: track 23.5 -> 37.0 mm
- net /SCL: track 42.3 -> 29.9 mm
- net /SDA: track 43.4 -> 34.0 mm, vias 2 -> 0
- net +3.3V: track 98.5 -> 107.2 mm, vias 3 -> 1
- net /BT_EN_3.3: track 80.5 -> 87.6 mm
- net /4.5_GEN: track 230.8 -> 225.9 mm
- net GND: track 9.29 -> 12.3 mm, vias 43 -> 38
- net /D+: track 74.2 -> 76.0 mm
Other:
- board text added: "3.3V"
- board text removed: "INT"
- board text removed: "OPT"
- board text removed: "VCC"

Commit message: stand 14:40 24.11.2025
Parts:
- added C3: 4.7µF, Capacitor_SMD:CP_Elec_4x5.4, B.Cu at (169.0, 77.4)
- added C4: 100nF, Capacitor_SMD:C_0805_2012Metric_Pad1.18x1.45mm_HandSolder, B.Cu at (164.2, 81.0)
- added C5: 100nF, Capacitor_SMD:C_0805_2012Metric_Pad1.18x1.45mm_HandSolder, B.Cu at (175.0, 101.2)
- added C6: 10µF, Capacitor_SMD:CP_Elec_4x5.4, B.Cu at (159.8, 94.8)
- added C7: 100nF, Capacitor_SMD:C_0805_2012Metric_Pad1.18x1.45mm_HandSolder, B.Cu at (168.6, 65.5)
- added C8: 100nF, Capacitor_SMD:C_0805_2012Metric_Pad1.18x1.45mm_HandSolder, B.Cu at (157.0, 67.2)
- added G***: LOGO, footprints:punti, B.Cu at (128.2, 78.2)
- added G***: LOGO, LOGO, B.Cu at (158.6, 86.4)
- C1: value 22u -> 22µF
- C2: value C_Small -> 100nF
- R1: value R -> 10k
Routing:
- net +3.3V: track 107.2 -> 113.9 mm
- net /4.5_GEN: track 225.9 -> 231.1 mm
- net /SDA: track 34.0 -> 34.8 mm
- net GND: vias 38 -> 36
Other:
- board text added: "1.3µH"
- board text added: "100nF"
- board text added: "10k"
- board text added: "10µF"
- board text added: "140k"
- board text added: "22µF"
- board text added: "30.9k"
- board text added: "4.7µF"
- board text added: "B+"
- board text added: "B-"
- board text added: "D-FF"
- board text added: "DC-DC"
- board text added: "LS"
