File: ruecklicht.kicad_sch (KiCad schematic)
At the start: 0 parts

Commit message: stand 15:32
Other:
- added sheet battery (schematic/battery.kicad_sch)
- added sheet leds (schematics/leds.kicad_sch)
- added sheet power_supply (schematics/power_supply.kicad_sch)
- added sheet switches (schematics/switches.kicad_sch)
- sheet ESP32 ports: added 3V3, GND; removed none

Commit message: stand ende 10.11.2025
Other:
- added sheet LS (schematics/ls.kicad_sch)
- sheet ESP32 ports: added BT_EN, D+; removed none
- sheet power_supply ports: added 4.5_IN; removed 4.5V, B+, B-
- sheet switches ports: added Q2; removed none

Commit message: 15.11.2025 15:12:00
Other:
- added sheet gyro (schematics/gyro.kicad_sch)
- sheet battery: file schematic/battery.kicad_sch -> schematics/battery.kicad_sch
Changed lines of the file:
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@@
 	(wire
 		(pts
-			(xy 66.04 64.77) (xy 66.04 53.34)
+			(xy 66.04 57.15) (xy 66.04 53.34)
 		)
 		(stroke
@@
 	(symbol
 		(lib_id "power:GND")
-		(at 66.04 64.77 0)
+		(at 66.04 57.15 0)
 		(unit 1)
 		(exclude_from_sim no)
@@
 		(fields_autoplaced yes)
 		(property "Reference" "#PWR07"
-			(at 66.04 71.12 0)
+			(at 66.04 63.5 0)
 			(effects
 				(font
@@
 		)
 		(property "Value" "GND"
-			(at 66.04 69.85 0)
+			(at 66.04 62.23 0)
 			(effects
 				(font
@@
 		)
 		(property "Footprint" ""
-			(at 66.04 64.77 0)
+			(at 66.04 57.15 0)
 			(effects
 				(font
@@
 		)
 		(property "Datasheet" ""
-			(at 66.04 64.77 0)
+			(at 66.04 57.15 0)
 			(effects
 				(font
@@
 		)
 		(property "Description" "Power symbol creates a global label with name \"GND\" , ground"
-			(at 66.04 64.77 0)
+			(at 66.04 57.15 0)
 			(effects
 				(font
@@
 			)
 		)
-		(property "Sheetfile" "schematic/battery.kicad_sch"
+		(property "Sheetfile" "schematics/battery.kicad_sch"
 			(at 25.4 37.4146 0)
 			(effects
@@
 				)
 			)
+		)
+	)
+	(sheet
+		(at 72.39 85.09)
+		(size 21.59 10.16)
+		(exclude_from_sim no)
+		(in_bom yes)
+		(on_board yes)
+		(dnp no)
+		(fields_autoplaced yes)
+		(stroke
+			(width 0.1524)
+			(type solid)
+		)
+		(fill
+			(color 0 0 0 0.0000)
+		)
+		(property "Sheetname" "gyro"
+			(at 72.39 84.3784 0)
+			(effects
+				(font
+					(size 1.27 1.27)
+				)
+				(justify left bottom)
+			)
+		)
+		(property "Sheetfile" "schematics/gyro.kicad_sch"
+			(at 72.39 95.8346 0)
+			(effects
+				(font
+					(size 1.27 1.27)
+				)
+				(justify left top)
+			)
+		)
+		(instances
+			(project "ruecklicht"
+				(path "/d9fee8f2-a86d-4098-a09f-80e037052314"
+					(page "9")
+				)
+			)

Commit message: 15.11.2025 16:38
Other:
- sheet gyro ports: added ADO, GND, INT, SCL, SDA, VDD; removed none

Commit message: 16.11.2025 13:36 -> Schematic Finished (possible)
Other:
- sheet ESP32 ports: added SCL, SDA; removed none
Changed lines of the file:
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@@
-	(wire
-		(pts
-			(xy 130.81 82.55) (xy 130.81 87.63)
-		)
-		(stroke
-			(width 0)
-			(type default)
-		)
-	)
 	(wire
 		(pts
@@
 	(wire
 		(pts
-			(xy 208.28 64.77) (xy 214.63 64.77)
+			(xy 204.47 64.77) (xy 214.63 64.77)
 		)
 		(stroke
@@
 	(wire
 		(pts
-			(xy 208.28 82.55) (xy 208.28 74.93)
+			(xy 204.47 82.55) (xy 204.47 74.93)
 		)
 		(stroke
@@
 	(wire
 		(pts
+			(xy 199.39 34.29) (xy 210.82 34.29)
+		)
+		(stroke
+			(width 0)
+			(type default)
+		)
+	)
+	(wire
+		(pts
 			(xy 101.6 33.02) (xy 115.57 33.02)
 		)
@@
 	(wire
 		(pts
-			(xy 208.28 74.93) (xy 214.63 74.93)
+			(xy 204.47 74.93) (xy 214.63 74.93)
 		)
 		(stroke
@@
 	(wire
 		(pts
-			(xy 208.28 69.85) (xy 214.63 69.85)
+			(xy 204.47 69.85) (xy 214.63 69.85)
 		)
 		(stroke
@@
 		(pts
 			(xy 199.39 41.91) (xy 210.82 41.91)
+		)
+		(stroke
+			(width 0)
+			(type default)
+		)
+	)
+	(wire
+		(pts
+			(xy 199.39 36.83) (xy 210.82 36.83)
 		)
 		(stroke
@@
 	)
 	(label "D+"
-		(at 208.28 69.85 0)
+		(at 204.47 69.85 0)
+		(effects
+			(font
+				(size 1.27 1.27)
+			)
+			(justify left bottom)
+		)
+	)
+	(label "4.5_GEN"
+		(at 130.81 87.63 0)
 		(effects
 			(font
@@
 		)
 	)
-	(label "LEDs"
-		(at 208.28 64.77 0)
-		(effects
-			(font
-				(size 1.27 1.27)
-			)
-			(justify left bottom)
-		)
-	)
 	(label "B+"
 		(at 66.04 24.13 180)
@@
 			)
 			(justify right bottom)
+		)
+	)
+	(label "4.5_GEN"
+		(at 204.47 64.77 0)
+		(effects
+			(font
+				(size 1.27 1.27)
+			)
+			(justify left bottom)
 		)
 	)
@@
 	(symbol
 		(lib_id "power:GND")
-		(at 208.28 82.55 0)
+		(at 204.47 82.55 0)
 		(unit 1)
 		(exclude_from_sim no)
@@
 		(fields_autoplaced yes)
 		(property "Reference" "#PWR08"
-			(at 208.28 88.9 0)
+			(at 204.47 88.9 0)
 			(effects
 				(font
@@
 		)
 		(property "Value" "GND"
-			(at 208.28 87.63 0)
+			(at 204.47 87.63 0)
 			(effects
 				(font
@@
 		)
 		(property "Footprint" ""
-			(at 208.28 82.55 0)
+			(at 204.47 82.55 0)
 			(effects
 				(font
@@
 		)
 		(property "Datasheet" ""
-			(at 208.28 82.55 0)
+			(at 204.47 82.55 0)
 			(effects
 				(font
@@
 		)
 		(property "Description" "Power symbol creates a global label with name \"GND\" , ground"
-			(at 208.28 82.55 0)
+			(at 204.47 82.55 0)
 			(effects
 				(font
@@
 	)
 	(symbol
-		(lib_id "power:+3.3VP")
-		(at 130.81 82.55 0)
-		(unit 1)
-		(exclude_from_sim no)
-		(in_bom yes)
-		(on_board yes)
-		(dnp no)
-		(fields_autoplaced yes)
-		(property "Reference" "#PWR09"
-			(at 134.62 83.82 0)
-			(effects
-				(font
-					(size 1.27 1.27)
-				)
-				(hide yes)
-			)
-		)
-		(property "Value" "4.5V"
-			(at 130.81 77.47 0)
-			(effects
-				(font
-					(size 1.27 1.27)
-				)
-			)
-		)
-		(property "Footprint" ""
-			(at 130.81 82.55 0)
-			(effects
-				(font
-					(size 1.27 1.27)
-				)
-				(hide yes)
-			)
-		)
-		(property "Datasheet" ""
-			(at 130.81 82.55 0)
-			(effects
-				(font
-					(size 1.27 1.27)
-				)
-				(hide yes)
-			)
-		)
-		(property "Description" "Power symbol creates a global label with name \"+3.3VP\""
-			(at 130.81 82.55 0)
-			(effects
-				(font
-					(size 1.27 1.27)
-				)
-				(hide yes)
-			)
-		)
-		(pin "1"
-		)
-		(instances
-			(project "ruecklicht"
-				(path "/d9fee8f2-a86d-4098-a09f-80e037052314"
-					(reference "#PWR09")
-					(unit 1)
-				)
-			)
-		)
-	)
-	(symbol
 		(lib_id "power:GND")
 		(at 45.72 34.29 90)
@@
 			(effects
 				(font
+					(size 1.27 1.27)
+				)
+				(justify left)
+			)
+		)
+		(pin "SCL" input
+			(at 210.82 36.83 180)
+			(effects
+				(font
+					(size 1.27 1.27)
+				)
+				(justify left)
+			)
+		)
+		(pin "SDA" input
+			(at 210.82 34.29 180)
+			(effects
+				(font

Commit message: stand before gyro change
Other:
- sheet gyro ports: added none; removed ADO, INT
Changed lines of the file:
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@@
-			)
-		)
-		(pin "ADO" input
-			(at 93.98 93.98 0)
-			(effects
-				(font
-					(size 1.27 1.27)
-				)
-				(justify right)
 			)
 		)
@@
 			)
 		)
-		(pin "INT" input
-			(at 93.98 91.44 0)
-			(effects
-				(font
-					(size 1.27 1.27)
-				)
-				(justify right)
-			)
-		)

Commit message: stand 14:40 24.11.2025
Other:
- company: (none) -> Rücklicht 4
- title: (none) -> Rücklicht
Changed lines of the file:
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@@
 	(generator_version "9.0")
 	(paper "A4")
+	(title_block
+		(title "Rücklicht")
+		(date "17.11.2025")
+		(rev "1.0")
+		(company "Rücklicht 4")
+		(comment 1 "Matteo Huber, Lukas Köppl")
+		(comment 2 "Matthias Ulz, Adam Bukovjan")
+		(comment 3 "Mathias Kornschober, Christian Hanschitz")
+		(comment 4 "Gregor Gierlinger, Julian Gradwohl")
+	)
 	(wire
 		(pts
@@
 	(wire
 		(pts
-			(xy 63.5 101.6) (xy 63.5 95.25)
+			(xy 66.04 101.6) (xy 66.04 95.25)
 		)
 		(stroke
@@
 	(wire
 		(pts
-			(xy 63.5 90.17) (xy 72.39 90.17)
-		)
-		(stroke
-			(width 0)
-			(type default)
-		)
-	)
-	(wire
-		(pts
-			(xy 63.5 82.55) (xy 72.39 82.55)
+			(xy 66.04 90.17) (xy 74.93 90.17)
+		)
+		(stroke
+			(width 0)
+			(type default)
+		)
+	)
+	(wire
+		(pts
+			(xy 66.04 82.55) (xy 74.93 82.55)
 		)
 		(stroke
@@
 	(wire
 		(pts
-			(xy 63.5 95.25) (xy 72.39 95.25)
-		)
-		(stroke
-			(width 0)
-			(type default)
-		)
-	)
-	(wire
-		(pts
-			(xy 63.5 87.63) (xy 72.39 87.63)
+			(xy 66.04 95.25) (xy 74.93 95.25)
+		)
+		(stroke
+			(width 0)
+			(type default)
+		)
+	)
+	(wire
+		(pts
+			(xy 66.04 87.63) (xy 74.93 87.63)
 		)
 		(stroke
@@
 	(wire
 		(pts
-			(xy 66.04 57.15) (xy 66.04 53.34)
+			(xy 66.04 60.96) (xy 66.04 53.34)
 		)
 		(stroke
@@
 	(wire
 		(pts
-			(xy 63.5 76.2) (xy 63.5 82.55)
+			(xy 66.04 76.2) (xy 66.04 82.55)
 		)
 		(stroke
@@
 	)
 	(label "SDA"
-		(at 63.5 87.63 0)
+		(at 66.04 87.63 0)
 		(effects
 			(font
@@
 	)
 	(label "SCL"
-		(at 63.5 90.17 0)
+		(at 66.04 90.17 0)
 		(effects
 			(font
@@
 	(symbol
 		(lib_id "power:GND")
-		(at 66.04 57.15 0)
+		(at 66.04 60.96 0)
 		(unit 1)
 		(exclude_from_sim no)
@@
 		(fields_autoplaced yes)
 		(property "Reference" "#PWR07"
-			(at 66.04 63.5 0)
+			(at 66.04 67.31 0)
 			(effects
 				(font
@@
 		)
 		(property "Value" "GND"
-			(at 66.04 62.23 0)
+			(at 66.04 66.04 0)
 			(effects
 				(font
@@
 		)
 		(property "Footprint" ""
-			(at 66.04 57.15 0)
+			(at 66.04 60.96 0)
 			(effects
 				(font
@@
 		)
 		(property "Datasheet" ""
-			(at 66.04 57.15 0)
+			(at 66.04 60.96 0)
 			(effects
 				(font
@@
 		)
 		(property "Description" "Power symbol creates a global label with name \"GND\" , ground"
-			(at 66.04 57.15 0)
+			(at 66.04 60.96 0)
 			(effects
 				(font
@@
 	(symbol
 		(lib_id "power:+3.3V")
-		(at 63.5 76.2 0)
+		(at 66.04 76.2 0)
 		(unit 1)
 		(exclude_from_sim no)
@@
 		(fields_autoplaced yes)
 		(property "Reference" "#PWR06"
-			(at 63.5 80.01 0)
+			(at 66.04 80.01 0)
 			(effects
 				(font
@@
 		)
 		(property "Value" "+3.3V"
-			(at 63.5 71.12 0)
+			(at 66.04 71.12 0)
 			(effects
 				(font
@@
 		)
 		(property "Footprint" ""
-			(at 63.5 76.2 0)
+			(at 66.04 76.2 0)
 			(effects
 				(font
@@
 		)
 		(property "Datasheet" ""
-			(at 63.5 76.2 0)
+			(at 66.04 76.2 0)
 			(effects
 				(font
@@
 		)
 		(property "Description" "Power symbol creates a global label with name \"+3.3V\""
-			(at 63.5 76.2 0)
+			(at 66.04 76.2 0)
 			(effects
 				(font
@@
 	(symbol
 		(lib_id "power:GND")
-		(at 63.5 101.6 0)
+		(at 66.04 101.6 0)
 		(unit 1)
 		(exclude_from_sim no)
@@
 		(fields_autoplaced yes)
 		(property "Reference" "#PWR03"
-			(at 63.5 107.95 0)
+			(at 66.04 107.95 0)
 			(effects
 				(font
@@
 		)
 		(property "Value" "GND"
-			(at 63.5 106.68 0)
+			(at 66.04 106.68 0)
 			(effects
 				(font
@@
 		)
 		(property "Footprint" ""
-			(at 63.5 101.6 0)
+			(at 66.04 101.6 0)
 			(effects
 				(font
@@
 		)
 		(property "Datasheet" ""
-			(at 63.5 101.6 0)
+			(at 66.04 101.6 0)
 			(effects
 				(font
@@
 		)
 		(property "Description" "Power symbol creates a global label with name \"GND\" , ground"
-			(at 63.5 101.6 0)
+			(at 66.04 101.6 0)
 			(effects
 				(font
@@
 	)
 	(sheet
-		(at 72.39 80.01)
+		(at 74.93 80.01)
 		(size 21.59 17.78)
 		(exclude_from_sim no)
@@
 		)
 		(property "Sheetname" "gyro"
-			(at 72.39 79.2984 0)
+			(at 74.93 79.2984 0)
 			(effects
 				(font
@@
 		)
 		(property "Sheetfile" "schematics/gyro.kicad_sch"
-			(at 72.39 98.3746 0)
+			(at 74.93 98.3746 0)
 			(effects
 				(font
@@
 		)
 		(pin "GND" input
-			(at 72.39 95.25 180)
+			(at 74.93 95.25 180)
 			(effects
 				(font
@@
 		)
 		(pin "SCL" input
-			(at 72.39 90.17 180)
+			(at 74.93 90.17 180)
 			(effects
 				(font
@@
 		)
 		(pin "SDA" input
-			(at 72.39 87.63 180)
+			(at 74.93 87.63 180)
 			(effects
 				(font
@@
 		)
 		(pin "VDD" input
-			(at 72.39 82.55 180)
-			(effects
-				(font
+			(at 74.93 82.55 180)
+			(effects
+				(font
