File: schematics/battery.kicad_sch (KiCad schematic)
At the start: 2 parts

Commit message: 15.11.2025 15:12:00
Parts:
- renumbered B+ to B+1, B- to B-1
Changed lines of the file:
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@@
 		(dnp no)
 		(fields_autoplaced yes)
-		(property "Reference" "B+"
+		(property "Reference" "B+1"
 			(at 97.155 58.42 0)
 			(effects
@@
 		)
 		(instances
-			(project ""
+			(project "ruecklicht"
 				(path "/d9fee8f2-a86d-4098-a09f-80e037052314/09dee91a-e093-485b-bf09-2d4af5472fae"
-					(reference "B+")
+					(reference "B+1")
 					(unit 1)
 				)
@@
 		(dnp no)
 		(fields_autoplaced yes)
-		(property "Reference" "B-"
+		(property "Reference" "B-1"
 			(at 97.155 71.12 0)
 			(effects
@@
 			(project "ruecklicht"
 				(path "/d9fee8f2-a86d-4098-a09f-80e037052314/09dee91a-e093-485b-bf09-2d4af5472fae"
-					(reference "B-")
+					(reference "B-1")
 					(unit 1)
 				)

Commit message: 15.11.2025 16:38
Parts:
- added B2+1, B2-1, B3+1, B3-1: Conn_01x01_Pin, Connector_Wire:SolderWire-1.5sqmm_1x01_D1.7mm_OD3.9mm, symbol Connector:Conn_01x01_Pin
- renumbered B+1 to B1+1, B-1 to B1-1
Connections:
- net B-: now also B3-1.1 (Pin_1); no longer B1-1.1 (Pin_1)
- new net: B1-1.1 (Pin_1), B2+1.1 (Pin_1)
- new net: B2-1.1 (Pin_1), B3+1.1 (Pin_1)
Other:
- moved on the sheet: B1+1, B1-1

Commit message: stand 14:40 24.11.2025
Other:
- company: (none) -> Rücklicht 4
- title: (none) -> Rücklicht
- moved on the sheet: B1+1, B1-1, B2+1, B2-1, B3+1, B3-1
