File: schematics/gyro.kicad_sch (KiCad schematic)
At the start: 0 parts

Commit message: 15.11.2025 16:38
Parts:
- added J2: Conn_01x08_Pin, symbol Connector:Conn_01x08_Pin
- added R4, R5: R_Small, Resistor_SMD:R_1206_3216Metric_Pad1.30x1.75mm_HandSolder, symbol Device:R_Small
Connections:
- new net ADO: J2.7 (Pin_7)
- new net GND: J2.2 (Pin_2)
- new net INT: J2.8 (Pin_8)
- new net SCL: J2.3 (Pin_3), R4.2
- new net SDA: J2.4 (Pin_4), R5.2
- new net VDD: J2.1 (Pin_1), R4.1, R5.1
- new net XCL: J2.6 (Pin_6)
- new net XDA: J2.5 (Pin_5)

Commit message: 15.11.2025 16:51
Parts:
- J2: footprint (none) -> Connector_PinHeader_2.54mm:PinHeader_1x08_P2.54mm_Vertical
Changed lines of the file:
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@@
 			)
 		)
-		(property "Footprint" ""
+		(property "Footprint" "Connector_PinHeader_2.54mm:PinHeader_1x08_P2.54mm_Vertical"
 			(at 121.92 83.82 0)
 			(effects

Commit message: Finished Rev.1 -> possible order
Parts:
- J2: footprint Connector_PinHeader_2.54mm:PinHeader_1x08_P2.54mm_Vertical -> footprints:mpu6050-self
Changed lines of the file:
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@@
 			)
 		)
-		(property "Footprint" "Connector_PinHeader_2.54mm:PinHeader_1x08_P2.54mm_Vertical"
+		(property "Footprint" "footprints:mpu6050-self"
 			(at 121.92 83.82 0)
 			(effects

Commit message: stand 14:40 24.11.2025
Other:
- company: (none) -> Rücklicht 4
- title: (none) -> Rücklicht
Changed lines of the file:
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@@
 	(generator_version "9.0")
 	(paper "A4")
+	(title_block
+		(title "Rücklicht")
+		(date "17.11.2025")
+		(rev "1.0")
+		(company "Rücklicht 4")
+		(comment 1 "Matteo Huber, Lukas Köppl")
+		(comment 2 "Matthias Ulz, Adam Bukovjan")
+		(comment 3 "Mathias Kornschober, Christian Hanschitz")
+		(comment 4 "Gregor Gierlinger, Julian Gradwohl")
+	)
 	(junction
 		(at 151.13 83.82)
