File: schematics/power_supply.kicad_sch (KiCad schematic)
At the start: 0 parts

Commit message: stand ende 10.11.2025
Parts:
- added C1: 22u, symbol Device:C_Small
- added L1: 1.3u, symbol Device:L
- added R2: 140k, symbol Device:R_Small
- added R3: 30.9k, symbol Device:R_Small
- added U2: MP2128DT-LF-P, SOT23_MP2128_MNP, symbol symbols:MP2128DT-LF-P
Connections:
- net 3.3V: now also C1.2, L1.1, R2.1
- net GND: now also C1.1, R3.2, U2.2 (GND)
- new net: L1.2, U2.3 (SW)
- new net: R2.2, R3.1, U2.5 (FB)
- new net 4.5_IN: U2.1 (EN), U2.4 (IN)

Commit message: 15.11.2025 15:12:00
Parts:
- C1: footprint (none) -> Capacitor_SMD:CP_Elec_4x5.4
- L1: footprint (none) -> footprints:4310LC132KEC
- R2, R3: footprint (none) -> Resistor_SMD:R_1206_3216Metric_Pad1.30x1.75mm_HandSolder
- U2: footprint SOT23_MP2128_MNP -> Package_TO_SOT_SMD:SOT-23-5_HandSoldering
Changed lines of the file:
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@@
 			)
 		)
-		(property "Footprint" ""
+		(property "Footprint" "footprints:4310LC132KEC"
 			(at 157.48 73.66 0)
 			(effects
@@
 			)
 		)
-		(property "Footprint" "SOT23_MP2128_MNP"
+		(property "Footprint" "Package_TO_SOT_SMD:SOT-23-5_HandSoldering"
 			(at 106.68 68.58 0)
 			(effects
@@
 			)
 		)
-		(property "Footprint" ""
+		(property "Footprint" "Resistor_SMD:R_1206_3216Metric_Pad1.30x1.75mm_HandSolder"
 			(at 166.37 60.96 0)
 			(effects
@@
 			)
 		)
-		(property "Footprint" ""
+		(property "Footprint" "Resistor_SMD:R_1206_3216Metric_Pad1.30x1.75mm_HandSolder"
 			(at 166.37 68.58 0)
 			(effects
@@
 			)
 		)
-		(property "Footprint" ""
+		(property "Footprint" "Capacitor_SMD:CP_Elec_4x5.4"
 			(at 172.72 68.58 0)
 			(effects

Commit message: stand 14:40 24.11.2025
Parts:
- added C3: 4.7µF, Capacitor_SMD:CP_Elec_4x5.4, symbol Device:C_Small
- added C4: 100nF, Capacitor_SMD:C_0805_2012Metric_Pad1.18x1.45mm_HandSolder, symbol Device:C_Small
- C1: value 22u -> 22µF
Connections:
- net 4.5_IN: now also C3.1, C4.1
- net GND: now also C3.2, C4.2
Other:
- company: (none) -> Rücklicht 4
- title: (none) -> Rücklicht
- moved on the sheet: C1, L1, R2, R3
