File: schematics/schematics/d-ff.kicad_sch (KiCad schematic)
At the start: 1 part, among them IC1 SN74HCS74QDYYRQ1

Commit message: 15.11.2025 15:12:00
Parts:
- IC1: footprint SOP50P326X110-14N -> footprints:SOP50P326X110-14N
Changed lines of the file:
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@@
 			)
 		)
-		(property "Footprint" "SOP50P326X110-14N"
+		(property "Footprint" "footprints:SOP50P326X110-14N"
 			(at 161.29 186.36 0)
 			(effects

Commit message: stand 14:40 24.11.2025
Other:
- company: (none) -> Rücklicht 4
- title: (none) -> Rücklicht
Changed lines of the file:
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@@
 	(generator_version "9.0")
 	(paper "A4")
+	(title_block
+		(title "Rücklicht")
+		(date "17.11.2025")
+		(rev "1.0")
+		(company "Rücklicht 4")
+		(comment 1 "Matteo Huber, Lukas Köppl")
+		(comment 2 "Matthias Ulz, Adam Bukovjan")
+		(comment 3 "Mathias Kornschober, Christian Hanschitz")
+		(comment 4 "Gregor Gierlinger, Julian Gradwohl")
+	)
 	(wire
 		(pts
